File: MCU_Datalogger.kicad_pcb (KiCad board)
At the start: 4 copper layers, 52.1 x 31.8 mm, 30 parts, among them J1 Conn_01x04_Pin, J2 Conn_01x09_Pin, J3 Conn_01x04_Pin, J4 Conn_02x03_Odd_Even, U1 DS1337S_, U2 24LC1025, U3 24LC1025, U4 ATMEGA328P-AU, Y1 32.768 KHz, Y2 16 MHz

Commit message: Improve PCB design, add images folder, and bom folder
Parts:
- moved C4 28.4 mm to (56.8, 43.3)
- moved D1 28.4 mm to (58.7, 29.3)
- moved H2 28.4 mm to (23.8, 52.1)
- moved H4 28.4 mm to (69.5, 52.1)
- moved J2 28.4 mm to (28.9, 50.2)
- moved J3 28.4 mm to (54.9, 50.2)
- moved R1 28.4 mm to (31.4, 47.1)
- moved R2 28.4 mm to (36.5, 47.1)
- moved R4 28.4 mm to (56.8, 38.2)
- moved R6 28.4 mm to (61.0, 38.2)
- moved U3 28.4 mm to (34.2, 36.3)
- moved U4 28.4 mm to (47.2, 37.8)
- moved Y1 28.4 mm to (26.3, 43.3)
- moved BT1 28.4 mm to (26.3, 32.5)
- moved C1 28.4 mm to (41.0, 29.3)
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Routing:
- net GND: track 48.8 -> 52.3 mm
- net Net-(U4-PB7): track 21.7 -> 25.2 mm
- net /SCK: track 87.3 -> 85.9 mm
- net /Vcc: track 54.3 -> 55.5 mm
- net Net-(U1-X2): track 6.81 -> 7.97 mm
- net Net-(U4-PB6): track 21.4 -> 20.3 mm
- net Net-(U1-~{INTA}): track 5.77 -> 6.81 mm
- net /RESET: track 22.6 -> 23.4 mm
- net /MISO: track 22.2 -> 23.0 mm
