File: MCU_Datalogger.kicad_sch (KiCad schematic)
At the start: 25 parts, among them U1 DS1337S_, U2 24LC1025, U3 24LC1025, U4 ATMEGA328P-AU, Y1 32.768 KHz, Y2 16 MHz

Commit message: Improve PCB design, add images folder, and bom folder
Connections:
- net Abc123: no longer names the net of C4.2, U4.20 (AREF)
Changed lines of the file:
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@@
 		)
 	)
-	(label "Abc123"
-		(at 193.04 27.94 0)
-		(effects
-			(font
-				(size 1.27 1.27)
-			)
-			(justify left bottom)
-		)
-	)
 	(label "D5"
 		(at 231.14 46.99 0)
@@
 		)
 		(instances
-			(project "MCU Datalogger"
+			(project "MCU_Datalogger"
 				(path "/832ad2a6-1a19-40c8-8feb-ef3c152c556c"
 					(reference "R4")
@@
 		)
 		(instances
-			(project "MCU Datalogger"
+			(project "MCU_Datalogger"
 				(path "/832ad2a6-1a19-40c8-8feb-ef3c152c556c"
 					(reference "H4")
@@
 		)
 		(instances
-			(project "MCU Datalogger"
+			(project "MCU_Datalogger"
 				(path "/832ad2a6-1a19-40c8-8feb-ef3c152c556c"
 					(reference "#FLG02")
@@
 		)
 		(instances
-			(project "MCU Datalogger"
+			(project "MCU_Datalogger"
 				(path "/832ad2a6-1a19-40c8-8feb-ef3c152c556c"
 					(reference "#PWR04")
@@
 		)
 		(instances
-			(project "MCU Datalogger"
+			(project "MCU_Datalogger"
 				(path "/832ad2a6-1a19-40c8-8feb-ef3c152c556c"
 					(reference "#FLG03")
@@
 		)
 		(instances
-			(project "MCU Datalogger"
+			(project "MCU_Datalogger"
 				(path "/832ad2a6-1a19-40c8-8feb-ef3c152c556c"
 					(reference "Y1")
@@
 		)
 		(instances
-			(project "MCU Datalogger"
+			(project "MCU_Datalogger"
 				(path "/832ad2a6-1a19-40c8-8feb-ef3c152c556c"
 					(reference "R6")
@@
 		)
 		(instances
-			(project "MCU Datalogger"
+			(project "MCU_Datalogger"
 				(path "/832ad2a6-1a19-40c8-8feb-ef3c152c556c"
 					(reference "#PWR01")
@@
 		)
 		(instances
-			(project "MCU Datalogger"
+			(project "MCU_Datalogger"
 				(path "/832ad2a6-1a19-40c8-8feb-ef3c152c556c"
 					(reference "C1")
@@
 		)
 		(instances
-			(project "MCU Datalogger"
+			(project "MCU_Datalogger"
 				(path "/832ad2a6-1a19-40c8-8feb-ef3c152c556c"
 					(reference "R5")
@@
 		)
 		(instances
-			(project "MCU Datalogger"
+			(project "MCU_Datalogger"
 				(path "/832ad2a6-1a19-40c8-8feb-ef3c152c556c"
 					(reference "R1")
@@
 		)
 		(instances
-			(project "MCU Datalogger"
+			(project "MCU_Datalogger"
 				(path "/832ad2a6-1a19-40c8-8feb-ef3c152c556c"
 					(reference "BT1")
@@
 		)
 		(instances
-			(project "MCU Datalogger"
+			(project "MCU_Datalogger"
 				(path "/832ad2a6-1a19-40c8-8feb-ef3c152c556c"
 					(reference "#PWR06")
@@
 		)
 		(instances
-			(project "MCU Datalogger"
+			(project "MCU_Datalogger"
 				(path "/832ad2a6-1a19-40c8-8feb-ef3c152c556c"
 					(reference "#FLG01")
@@
 		)
 		(instances
-			(project "MCU Datalogger"
+			(project "MCU_Datalogger"
 				(path "/832ad2a6-1a19-40c8-8feb-ef3c152c556c"
 					(reference "#PWR07")
@@
 		)
 		(instances
-			(project "MCU Datalogger"
+			(project "MCU_Datalogger"
 				(path "/832ad2a6-1a19-40c8-8feb-ef3c152c556c"
 					(reference "U1")
@@
 		)
 		(instances
-			(project "MCU Datalogger"
+			(project "MCU_Datalogger"
 				(path "/832ad2a6-1a19-40c8-8feb-ef3c152c556c"
 					(reference "C5")
@@
 		)
 		(instances
-			(project "MCU Datalogger"
+			(project "MCU_Datalogger"
 				(path "/832ad2a6-1a19-40c8-8feb-ef3c152c556c"
 					(reference "D2")
@@
 		)
 		(instances
-			(project "MCU Datalogger"
+			(project "MCU_Datalogger"
 				(path "/832ad2a6-1a19-40c8-8feb-ef3c152c556c"
 					(reference "#PWR03")
@@
 		)
 		(instances
-			(project "MCU Datalogger"
+			(project "MCU_Datalogger"
 				(path "/832ad2a6-1a19-40c8-8feb-ef3c152c556c"
 					(reference "D1")
@@
 		)
 		(instances
-			(project "MCU Datalogger"
+			(project "MCU_Datalogger"
 				(path "/832ad2a6-1a19-40c8-8feb-ef3c152c556c"
 					(reference "C3")
@@
 		)
 		(instances
-			(project "MCU Datalogger"
+			(project "MCU_Datalogger"
 				(path "/832ad2a6-1a19-40c8-8feb-ef3c152c556c"
 					(reference "C2")
@@
 		)
 		(instances
-			(project "MCU Datalogger"
+			(project "MCU_Datalogger"
 				(path "/832ad2a6-1a19-40c8-8feb-ef3c152c556c"
 					(reference "R3")
@@
 		)
 		(instances
-			(project "MCU Datalogger"
+			(project "MCU_Datalogger"
 				(path "/832ad2a6-1a19-40c8-8feb-ef3c152c556c"
 					(reference "H3")
@@
 		)
 		(instances
-			(project "MCU Datalogger"
+			(project "MCU_Datalogger"
 				(path "/832ad2a6-1a19-40c8-8feb-ef3c152c556c"
 					(reference "U2")
@@
 		)
 		(instances
-			(project "MCU Datalogger"
+			(project "MCU_Datalogger"
 				(path "/832ad2a6-1a19-40c8-8feb-ef3c152c556c"
 					(reference "#PWR02")
@@
 		)
 		(instances
-			(project "MCU Datalogger"
+			(project "MCU_Datalogger"
 				(path "/832ad2a6-1a19-40c8-8feb-ef3c152c556c"
 					(reference "R2")
@@
 		)
 		(instances
-			(project "MCU Datalogger"
+			(project "MCU_Datalogger"
 				(path "/832ad2a6-1a19-40c8-8feb-ef3c152c556c"
 					(reference "H2")
@@
 		)
 		(instances
-			(project "MCU Datalogger"
+			(project "MCU_Datalogger"
 				(path "/832ad2a6-1a19-40c8-8feb-ef3c152c556c"
 					(reference "H1")
@@
 		)
 		(instances
-			(project "MCU Datalogger"
+			(project "MCU_Datalogger"
 				(path "/832ad2a6-1a19-40c8-8feb-ef3c152c556c"
 					(reference "U3")
@@
 		)
 		(instances
-			(project "MCU Datalogger"
+			(project "MCU_Datalogger"
 				(path "/832ad2a6-1a19-40c8-8feb-ef3c152c556c"
 					(reference "#PWR05")
@@
 		)
 		(instances
-			(project "MCU Datalogger"
+			(project "MCU_Datalogger"
 				(path "/832ad2a6-1a19-40c8-8feb-ef3c152c556c"
 					(reference "C4")
@@
 		)
 		(instances
-			(project "MCU Datalogger"
+			(project "MCU_Datalogger"
 				(path "/832ad2a6-1a19-40c8-8feb-ef3c152c556c"
 					(reference "U4")
@@
 		)
 		(instances
-			(project "MCU Datalogger"
+			(project "MCU_Datalogger"
 				(path "/832ad2a6-1a19-40c8-8feb-ef3c152c556c"
 					(reference "Y2")
@@
 		)
 		(instances
-			(project "MCU Datalogger"
+			(project "MCU_Datalogger"
 				(path "/832ad2a6-1a19-40c8-8feb-ef3c152c556c"
 					(reference "R7")
@@
 		)
 		(instances
-			(project "MCU Datalogger"
+			(project "MCU_Datalogger"
 				(path "/832ad2a6-1a19-40c8-8feb-ef3c152c556c"
 					(page "2")
